File: hardware/controller/kicad/controller-core-reva.kicad_sch (KiCad schematic)
At the start: 187 parts, among them J101 12V_ISOLATED_INPUT / JST XH, J102 STM_SWD / 1x6 2.54mm, J103 ESP_UART / 1x6 2.54mm, J104 UI_LINK / IDC 2x8 2.54mm, J105 JP13 NTC / 2 vías, J106 JP5 FLOW ADAPTER / VCC-GND-OC, J107 JP14 DOOR / contacto seco, J108 JP16 VISUAL V1..V8 / XH-8, J109 JP22 WATER / RED-WHITE-BLACK, J110 USB-C SERVICE / USB 2.0, J111 USB BENCH POWER / OPEN, J112 24V_ACTUATOR_INPUT / JST XH, J113 JP3 VALVE / JST XH, J114 POWER MONITOR / MEASURE ONLY, J115 JP8 GRINDER / 320VDC, J116 JP19 HEATER / 1900W 27R5, J117 JP24 PUMP / 230VAC, J118 JP17 MAINS / L-N, J119 JP1 PE TO BOILER, J120 JP9 PE INPUT, J121 24V INTERNAL SELECT / OPEN FO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, K701 G5RL-1A-E-TV8 DC24, Q501 SI2308A, Q701 SI2308A / relay coil, Q703 BTA24-800BWRG / heater, Q704 BTA24-800BWRG / pump, Q705 SI2308A / heater opto LED, Q706 SI2308A / pump opto LED, Q707 SI2308A / grinder opto LED, Q708 BTA24-800BWRG / grinder, U101 STM32G431RBT6, U201 ESP32-S3-WROOM-1U-N8R8, U203 USBLC6-2SC6, U301 AP63203WU-7, U302 TPS22918DBVR, U303 AP63200WU-7 / 24V to 12V, U501 DRV8876PWPR, U502 UCC27517DBVR, U601 TPS3828-33DBVR, U602 SN74LVC2G08DCTR, U603 SN74LVC2G08DCTR, U604 SN74LVC2G08DCTR, U701 MOC3083 / zero-cross, U702 MOC3083 / zero-cross, U703 MOC3083 / zero-cross

Commit message: Add ground fills, silkscreen, per-device mains rules, USB pair and TE FASTON tabs
Fills: on the owner's delegation, F.Cu and B.Cu carry GND_UI over the whole
SELV side, with the inner planes' outline, stitched to In1.Cu by 156 vias
of 0.6 mm on a 5 mm grid wherever they clear copper, courtyards and
keepouts. SMD pads join solid, through-hole pads with reliefs; one spoke is
accepted on ground pads, which also meet the plane. 0.5 mm of clearance
keeps the USB pair near its impedance. The mains side gets no fill.

Silkscreen: a new script draws the owner's logo (traced from bicho.png),
the title, every harness and service connector's original JP name and
function, + and - on JP8, L and N on JP17, and a mains warning in the
copper-free barrier band. Labels are placed automatically clear of pads,
silkscreen and courtyards, with JP8, JP17, JP19 and JP21 fixed by hand. A
second script exports a 1:1 PDF shifted off the page corner with a 100 mm
scale bar for the paper check.

Optocouplers: the device-pitch and slot areas all shared one name, so the
0.6 mm and 6 mm relaxations also applied between items of different
devices. Each area is now named after its part with a rule of its own; the
one real case it exposed, the B.Cu drop to Q708 at 1.3 mm from the grinder
gate, now stops in the top of the pad. The slot gives about 9 mm of surface
path and 6.02 mm of air.

USB: the JLCPCB calculator for JLC04161H-7628 gives 90 ohm differential
at 0.29 mm with a 0.20 mm gap; 0.20/0.20 was about 104 ohm. The U203 to
R221/R222 run is coupled that way and the class rule follows.

JP1/JP9: the owner's photo shows vertical two-leg tabs, matched to TE
63824-1 (C575074): two 1.40 mm holes at 5.08 mm per TE's drawing. The PE
bond is four 3 mm runs and each tab's legs are linked.

ERC 0, netlist 187 components / 612 pins. DRC with all severities: no
violations, no open connections, the three mounting-hole parity entries.

Co-Authored-By: Claude Opus 5.5 <noreply@anthropic.com>
Parts:
- J119, J120: footprint OpenSaeco:FASTON_Tab_6.3x0.8mm_PE -> OpenSaeco:TE_FASTON_63824-1_Tab_6.35mm_Vertical; jlc_class (none) -> Extended; lcsc (none) -> C575074; manufacturer (none) -> TE Connectivity; mpn (none) -> 63824-1; pcba_type (none) -> TBD

Commit message: Fit JP17 with its TE RAST 5 header and flag the unmatched harness housings
The owner read TE 2-1241961-7 on the JP17 harness housing, a RAST 5
receptacle with 1b polarization, so J118 moves from a JST B3P-VH to the
matching TE 1971845-3 (LCSC C5169636). Its footprint follows TE drawing
C-1971845 for an odd number of tabs, with J116's convention. It sits flush
with the bottom edge, 2.5 mm west of the photographed centre, so the PS701
neutral climbs between the polarizing post and the PE tabs. Phase, neutral
and silkscreen around it are rerouted; DRC stays clean.

Re-reading the caliper photos against JST's drawings shows the signal
housings are narrower than XH/PH and JP24/JP8 wider than VH. Those
footprints stay as placeholders, now marked as such in the docs.

Co-Authored-By: Claude Opus 5.5 <noreply@anthropic.com>
Parts:
- J118: footprint Connector_JST:JST_VH_B3P-VH_1x03_P3.96mm_Vertical -> OpenSaeco:TE_RAST5_1971845-3_1x03_P5.00mm_Vertical; lcsc C160316 -> C5169636; manufacturer JST -> TE Connectivity; mpn B3P-VH(LF)(SN) -> 1971845-3

Commit message: Fit the owner-identified HR A2506 and LEOCO harness headers
The owner confirmed the headers the original harness housings mate with.
JP3, JP5 and JP13 are HR (Joint Tech) A2506WV-05P/-03P/-02P (LCSC C382535,
C382533, C382532), not JST XH. JP8 and JP24 are LEOCO 3941P03*000 (3.96 mm)
and 5001P020013 (5.00 mm), which JLCPCB does not stock, so they carry no LCSC
code and are hand-soldered or consigned.

Five footprints are drawn from the makers' drawings (A2506WV-XP rev B5,
394105S rev F, 500101S rev D), with pad 1 on each drawing's circuit 1. The
A2506 keeps the XH pad row, so J105, J113 and their copper stay put; J106
moves 0.3 mm west so its deeper housing clears U702. J115 keeps the VH row
with 1.80 mm holes. J117 goes to a 5 mm pitch, centred 0.5 mm east of the
photographed JP24 to clear JP19; its neutral leaves the south half of pin 2
to hold 2.5 mm from the phase. The JP17 L mark moves east of tab 1.

The checker accepts owner-identified parts with zero stock or no JLCPCB code
when the catalog says so explicitly. The print export now finds kicad-cli on
Windows. ERC 0, netlist 187/612; DRC with all severities: 0 violations,
0 unconnected, parity only MH1-MH3. The stock freshness gate still fails on
untouched parts checked more than 7 days ago. The JP8 hook orientation, which
sets the grinder polarity, must be checked against the harness.

Co-Authored-By: Claude Opus 5.5 <noreply@anthropic.com>
Parts:
- J105: footprint Connector_JST:JST_XH_B2B-XH-A_1x02_P2.50mm_Vertical -> OpenSaeco:HR_A2506WV-02P_1x02_P2.50mm_Vertical; lcsc C158012 -> C382532; manufacturer JST -> HR(Joint Tech Elec); mpn B2B-XH-A(LF)(SN) -> A2506WV-02P
- J106: footprint Connector_JST:JST_XH_B3B-XH-A_1x03_P2.50mm_Vertical -> OpenSaeco:HR_A2506WV-03P_1x03_P2.50mm_Vertical; lcsc C144394 -> C382533; manufacturer JST -> HR(Joint Tech Elec); mpn B3B-XH-A(LF)(SN) -> A2506WV-03P
- J113: value JP3 VALVE / JST XH -> JP3 VALVE / A2506; footprint Connector_JST:JST_XH_B5B-XH-A_1x05_P2.50mm_Vertical -> OpenSaeco:HR_A2506WV-05P_1x05_P2.50mm_Vertical; lcsc C157991 -> C382535; manufacturer JST -> HR(Joint Tech Elec); mpn B5B-XH-A(LF)(SN) -> A2506WV-05P
- J115: footprint Connector_JST:JST_VH_B3P-VH_1x03_P3.96mm_Vertical -> OpenSaeco:LEOCO_3941P03_1x03_P3.96mm_Vertical; jlc_class Extended -> (none); lcsc C160316 -> (none); manufacturer JST -> LEOCO; mpn B3P-VH(LF)(SN) -> 3941P03*000; pcba_type TBD -> hand_solder_or_consigned
- J117: footprint Connector_JST:JST_VH_B2P-VH_1x02_P3.96mm_Vertical -> OpenSaeco:LEOCO_5001P02_1x02_P5.00mm_Vertical; jlc_class Extended -> (none); lcsc C160315 -> (none); manufacturer JST -> LEOCO; mpn B2P-VH(LF)(SN) -> 5001P020013; pcba_type TBD -> hand_solder_or_consigned
Other:
- note added: "10 / Entradas pasivas — JP13 y JP5 HR A2506; resto, huellas candidatas por foto"
- note removed: "10 / Entradas pasivas — huellas candidatas según fotos con calibre"
