File: hardware/front-panel/kicad/front-panel-reva.kicad_sch (KiCad schematic)
At the start: 44 parts, among them J1 UI_LINK / IDC 2x8 2.54mm, J2 LCD_ADAPTER / 8 pins, SW1 KEY 1 / NO, SW2 KEY 2 / NO, SW3 KEY 3 / NO, SW4 KEY 4 / NO, SW5 KEY 5 / NO, SW6 KEY 6 / NO, SW7 KEY 7 / NO, SW8 KEY 8 / NO, U1 TCA9534PWR

Commit message: Lay out and route the front panel PCB for JLCPCB
Assign JLC parts to the open positions: HRO K2-1102SP-A4SC-04 6x6x4.3 mm
switches (C83916) with a project footprint from the EasyEDA land pattern,
JST S8B-PH-K-S for J2 in the Waveshare cable order (C157915), and the
standby LED on TCA9534 P7 (KT-0603R + 470R). Seven key channels replace
the eighth, whose parts are removed from schematic and board.

layout_front_panel_pcb.py places the parts on the measured positions,
routes with Freerouting 2.4.1 through Specctra DSN/SES and pours GND on
both layers with stitching and island anchoring. KiCad 10.0.6 DRC with
schematic parity and all severities: 0 violations, 0 unconnected, 0
parity issues. export_front_panel_fab.py writes Gerbers, drill, BOM and
CPL for JLCPCB; the package stays a candidate pending the checks listed
in hardware/front-panel/layout.md.

Co-Authored-By: Claude Opus 5 <noreply@anthropic.com>
Parts:
- removed C18: 100nF / filtro, Capacitor_SMD:C_0603_1608Metric, symbol OpenSaeco:C
- removed R18: 10k / pull-up, Resistor_SMD:R_0603_1608Metric, symbol OpenSaeco:R
- removed R28: 1k / serie, Resistor_SMD:R_0603_1608Metric, symbol OpenSaeco:R
- removed SW8: KEY 8 / NO, symbol OpenSaeco:SW
- added D1: KT-0603R / STBY, LED_SMD:LED_0603_1608Metric, symbol OpenSaeco:LED
- added R7: 470 / LED, Resistor_SMD:R_0603_1608Metric, symbol OpenSaeco:R
- J2: value LCD_ADAPTER / 8 pins -> LCD_ADAPTER / JST PH 8; footprint (none) -> Connector_JST:JST_PH_S8B-PH-K_1x08_P2.00mm_Horizontal; jlc_class (none) -> Extended; lcsc (none) -> C157915; manufacturer (none) -> JST; mpn (none) -> S8B-PH-K-S(LF)(SN); pcba_type (none) -> Economic and Standard
- SW1: value KEY 1 / NO -> KEY 1 / PB1; footprint (none) -> OpenSaeco:SW_HRO_K2-1102SP-A4SC-04; jlc_class (none) -> Extended; lcsc (none) -> C83916; manufacturer (none) -> Korean Hroparts Elec; mpn (none) -> K2-1102SP-A4SC-04; pcba_type (none) -> Economic and Standard
- SW2: value KEY 2 / NO -> KEY 2 / PB2; footprint (none) -> OpenSaeco:SW_HRO_K2-1102SP-A4SC-04; jlc_class (none) -> Extended; lcsc (none) -> C83916; manufacturer (none) -> Korean Hroparts Elec; mpn (none) -> K2-1102SP-A4SC-04; pcba_type (none) -> Economic and Standard
- SW3: value KEY 3 / NO -> KEY 3 / PB3; footprint (none) -> OpenSaeco:SW_HRO_K2-1102SP-A4SC-04; jlc_class (none) -> Extended; lcsc (none) -> C83916; manufacturer (none) -> Korean Hroparts Elec; mpn (none) -> K2-1102SP-A4SC-04; pcba_type (none) -> Economic and Standard
- SW4: value KEY 4 / NO -> KEY 4 / PB8; footprint (none) -> OpenSaeco:SW_HRO_K2-1102SP-A4SC-04; jlc_class (none) -> Extended; lcsc (none) -> C83916; manufacturer (none) -> Korean Hroparts Elec; mpn (none) -> K2-1102SP-A4SC-04; pcba_type (none) -> Economic and Standard
- SW5: value KEY 5 / NO -> KEY 5 / PB4/PB6; footprint (none) -> OpenSaeco:SW_HRO_K2-1102SP-A4SC-04; jlc_class (none) -> Extended; lcsc (none) -> C83916; manufacturer (none) -> Korean Hroparts Elec; mpn (none) -> K2-1102SP-A4SC-04; pcba_type (none) -> Economic and Standard
- SW6: value KEY 6 / NO -> KEY 6 / PB5; footprint (none) -> OpenSaeco:SW_HRO_K2-1102SP-A4SC-04; jlc_class (none) -> Extended; lcsc (none) -> C83916; manufacturer (none) -> Korean Hroparts Elec; mpn (none) -> K2-1102SP-A4SC-04; pcba_type (none) -> Economic and Standard
- SW7: value KEY 7 / NO -> KEY 7 / PB7; footprint (none) -> OpenSaeco:SW_HRO_K2-1102SP-A4SC-04; jlc_class (none) -> Extended; lcsc (none) -> C83916; manufacturer (none) -> Korean Hroparts Elec; mpn (none) -> K2-1102SP-A4SC-04; pcba_type (none) -> Economic and Standard
Connections:
- net 3V3_UI: now also R7.1
- net KEY_8_N renamed LED_STBY_N
- net LED_STBY_N: now also D1.1 (K)
- new net LED_STBY_A: D1.2 (A), R7.2
Other:
- note added: "05 / Siete pulsadores en las posiciones originales; P7 enciende el LED STBY (activo a 0)"
- note added: "100nF: X7R; 1uF/10uF: X5R, temperatura y DC bias pendientes. SW: HRO K2-1102SP-A4SC-04, 6x6x4,3 mm."
- note added: "Contorno y pulsadores según hardware/front-panel/mechanical.md. Borrador en revisión. Validación: tools/validate_kicad.py."
- note added: "LED: 3V3 - R7 - D1 - P7. P7 arranca como entrada: LED apagado hasta configurarlo."
- note added: "Orden del cable PH 2,0 del módulo Waveshare 2": VCC GND DIN CLK CS DC RST BL."
- note removed: "05 / Ocho canales previstos — cantidad y mecánica originales pendientes"
- note removed: "100nF: X7R; 1uF/10uF: X5R, temperatura y DC bias pendientes. J2 y SW1–SW8 sin huella."
- note removed: "Sin contorno ni posición real de botones. No fabricar. Validación: tools/validate_kicad.py."

Commit message: Enter every harness connector from the top
The owner wants every wire-to-board header vertical, to free the board
area the side-entry housings took. The JST S-series headers become their
B-series twins: B2B-XH-A on J101, J105, J107 and J112, B3B-XH-A on J106,
B5B-XH-A on J113, B8B-XH-A on J108, B3B-PH-K-S on J109, B2P-VH on J117,
B3P-VH on J115 and J118, and B8B-PH-K-S on the front panel's J2. All are
in stock at JLCPCB; the assembly type is still to be confirmed.

KiCad's footprints for both series share pad position, pitch and drill,
so each part keeps its origin and rotation and the copper is untouched.
The one exception is J118: the vertical VH housing reaches 4.2 mm north
of its pins and hit PS701's courtyard by 0.6 mm, so it drops 0.8 mm, well
within JP17's 1.5 mm tolerance, and its three track stubs follow.

The courtyards give back about 750 mm2 on the main board, the useful part
beside J107/J108 and under J101/J112. ERC is clean on both boards. The
main board's DRC is unchanged: two intentional dangling ends, 77 open
connections and the three mounting-hole parity notes. The front panel
has no violations once its ground pour is refilled.

Co-Authored-By: Claude Opus 5 <noreply@anthropic.com>
Parts:
- J2: footprint Connector_JST:JST_PH_S8B-PH-K_1x08_P2.00mm_Horizontal -> Connector_JST:JST_PH_B8B-PH-K_1x08_P2.00mm_Vertical; lcsc C157915 -> C157974; mpn S8B-PH-K-S(LF)(SN) -> B8B-PH-K-S(LF)(SN); pcba_type Economic and Standard -> TBD

Commit message: Fit the owner-identified Wurth WR-MM front-panel link on both boards
The owner identified the connector of the original link between the main
board and the front panel as Wurth WR-MM 690367181672 (16 contacts at
1.27 mm stagger), the same part at both ends of a 1:1 16-wire flat cable.
The latch of the cable plug enters a 1.5 mm hole beside pin 1, which locks
it and sets its direction, so pin 1 always meets pin 1. It replaces the
2x8 IDC in J104 and J1. JLCPCB lists it as C19103863, without stock.

The footprint follows Wurth drawing 690367181672 rev 002.000: 0.85 mm
holes, 1.4 mm pads, a 22.32 x 5 mm body and the 1.5 mm non-plated latch
hole; it gets a 6.1 mm tall stand-in model shared by both boards.

- Main board: J104 turns 180 deg with pin 1 on the IDC's pin 1, so the
  odd pins stay and the even pins move 1.27 mm east. 3V3_UI passes west of
  the latch hole; DC, BL and SDA reach their new pins and SCL and INT end on
  the pad centres. 1315 segments, 439 vias.
- Front panel: J1 is centred on the original JP3 zone, C3 stays by pin 1,
  rerouted by Freerouting (297 segments, 192 vias); fab package refreshed.

The photo count of 20 contacts for JP21 was wrong. ERC 0 on both boards;
netlists 187/612 and 42/118. DRC with all severities: main 0 violations,
0 unconnected, parity only MH1-MH3; front 0/0/0. Still to do: try the
cable latch in both new boards; 3V3_UI rides one 1.5 A contact.

Co-Authored-By: Claude Opus 5.5 <noreply@anthropic.com>
Parts:
- J1: value UI_LINK / IDC 2x8 2.54mm -> UI_LINK / WR-MM 16; footprint Connector_IDC:IDC-Header_2x08_P2.54mm_Vertical -> OpenSaeco:Wurth_WR-MM_690367181672_2x08_P1.27mm_Vertical; lcsc C7501244 -> C19103863; manufacturer Megastar -> Wurth Elektronik; mpn ZX-IDC2.54-2-8PZZ -> 690367181672; pcba_type Economic and Standard -> TBD
Other:
- note added: "J1: WR-MM del JP3 original; pinout nuevo, no el Saeco."
- note removed: "J1 NO corresponde a JP21 Saeco."
